Commit message: updated .xacro (and .gazebo-as-xacro) files in p3dx_description to newer Gazebo and xacro standards, including 'xacro:' additions and a material-color-fix due to a problematic property ('name=') in the 'visual' tag; updated directory names to correspond to the package names in CMakeLists.txt and package.xml

File: p3dx_description_mod/urdf/pioneer3dx.xacro (robot description, xacro)
@@ -16,4 +16,10 @@
 work original in ucs-ros-pkg.
  -->
+<!-- ...if needed, for completeness and file-checking...
+create xml file from xacro file(s) via:
+$ rosrun xacro xacro pioneer3dx.xacro > pioneer3dx.xml
+create inorder processing version via:
+$ rosrun xacro xacro -i pioneer3dx.xacro > pioneer3dx.xml
+-->
 <robot name="pioneer3dx" xmlns:xacro="http://ros.org/wiki/xacro">
   <!-- import all gazebo-customization elements, including gazebo colors -->
@@ -29,5 +35,6 @@
 			<inertia ixx="1" ixy="0" ixz="0" iyy="1" iyz="0" izz="1" />
 		</inertial>
-		<visual name="base_visual">
+		<!-- <visual name="base_visual"> name tag throws off parser in Gazebo 5+ when dealing with colors, removing... -->
+        <visual>
 			<origin xyz="-0.045 0 0.148" rpy="0 0 0" />
 			<geometry name="pioneer_geom">
@@ -52,5 +59,6 @@
 			<inertia ixx="1" ixy="0" ixz="0" iyy="1" iyz="0" izz="1" />
 		</inertial>
-		<visual name="base_visual">
+		<!-- <visual name="base_visual"> name tag throws off parser in Gazebo 5+ when dealing with colors, removing... -->
+        <visual>
 			<origin xyz="0 0 0" rpy="0 0 0" />
 			<geometry name="top_geom">
@@ -80,5 +88,6 @@
 			<inertia ixx="0.01" ixy="0" ixz="0" iyy="0.01" iyz="0" izz="0.01" />
 		</inertial>
-		<visual name="base_visual">
+		<!-- <visual name="base_visual"> name tag throws off parser in Gazebo 5+ when dealing with colors, removing... -->
+        <visual>
 			<origin xyz="0 0 0" rpy="0 0 0" />
 			<geometry name="pioneer_geom">
@@ -113,5 +122,6 @@
 				iyy="0.015218160428" iyz="-0.000004273467" izz="0.011763977943" />
 		</inertial>
-		<visual name="base_visual">
+		<!-- <visual name="base_visual"> name tag throws off parser in Gazebo 5+ when dealing with colors, removing... -->
+        <visual>
 			<origin xyz="0 0 0" rpy="0 0 0" />
 			<geometry name="pioneer_geom">
@@ -146,5 +156,6 @@
 				iyy="0.015218160428" iyz="-0.000004273467" izz="0.011763977943" />
 		</inertial>
-		<visual name="base_visual">
+		<!-- <visual name="base_visual"> name tag throws off parser in Gazebo 5+ when dealing with colors, removing... -->
+        <visual>
 			<origin xyz="0 0 0" rpy="0 0 0" />
 			<geometry name="pioneer_geom">
@@ -176,5 +187,6 @@
 			<inertia ixx="1" ixy="0" ixz="0" iyy="1" iyz="0" izz="1" />
 		</inertial>
-		<visual name="front_sonar_vis">
+		<!-- <visual name="front_sonar_vis"> name tag throws off parser in Gazebo 5+ when dealing with colors, removing... -->
+        <visual>
 			<origin rpy="0 0 0" xyz="0 0 0" />
 			<geometry name="pioneer_geom">

File: p3dx_description_mod/urdf/pioneer3dx_wheel.xacro (robot description, xacro)
@@ -17,6 +17,7 @@
  -->
 <robot xmlns:xacro="http://ros.org/wiki/xacro">
-	<!-- properties (constants) -->
-	<property name="M_PI" value="3.14159" />
+    <!-- properties (constants) -->
+	<!-- <xacro:property name="M_PI" value="3.14159" /> -->
+    <xacro:property name="M_PI" value="3.14159" />
 	<!-- right/left hubcap + wheel -->
 	<xacro:macro name="p3dx_wheel" params="suffix parent reflect">
@@ -29,5 +30,6 @@
 					iyz="0" izz="0.011763977943" />
 			</inertial>
-			<visual name="base_visual">
+			<!-- <visual name="base_visual"> name tag throws off parser in Gazebo 5+ when dealing with colors, removing... -->
+            <visual>
 				<origin xyz="0 0 0" rpy="0 0 0" />
 				<geometry name="pioneer_geom">
@@ -59,5 +61,6 @@
 					iyz="0" izz="0.011763977943" />
 			</inertial>
-			<visual name="base_visual">
+			<!-- <visual name="base_visual"> name tag throws off parser in Gazebo 5+ when dealing with colors, removing... -->
+            <visual>
 				<origin xyz="0 0 0" rpy="0 0 0" />
 				<geometry name="pioneer_geom">
