Commit message: fixing internal naming (base_link_*_wheel_joint instead of base_*_wheel_joint); adding default parameters for DiffDrive

File: p3dx_description/urdf/pioneer3dx.xacro (robot description, xacro)
@@ -18,7 +18,7 @@
 <robot name="pioneer3dx" xmlns:xacro="http://ros.org/wiki/xacro">
   <!-- import all gazebo-customization elements, including gazebo colors -->
-  <xacro:include filename="$(find p3dx_description)/urdf/pioneer3dx.gazebo" />
+  <xacro:include filename="$(find p3dx_description_mod)/urdf/pioneer3dx.gazebo" />
   <!-- import the pioneer 3dx's wheels -->
-  <xacro:include filename="$(find p3dx_description)/urdf/pioneer3dx_wheel.xacro" />
+  <xacro:include filename="$(find p3dx_description_mod)/urdf/pioneer3dx_wheel.xacro" />
   <!-- chassis -->
 	<link name="base_link">
@@ -32,5 +32,5 @@
 			<origin xyz="-0.045 0 0.148" rpy="0 0 0" />
 			<geometry name="pioneer_geom">
-				<mesh filename="package://p3dx_description/meshes/chassis.stl" />
+				<mesh filename="package://p3dx_description_mod/meshes/chassis.stl" />
 			</geometry>
 			<material name="ChassisRed">
@@ -55,5 +55,5 @@
 			<origin xyz="0 0 0" rpy="0 0 0" />
 			<geometry name="top_geom">
-				<mesh filename="package://p3dx_description/meshes/top.stl" />
+				<mesh filename="package://p3dx_description_mod/meshes/top.stl" />
 			</geometry>
 			<material name="TopBlack">
@@ -83,5 +83,5 @@
 			<origin xyz="0 0 0" rpy="0 0 0" />
 			<geometry name="pioneer_geom">
-				<mesh filename="package://p3dx_description/meshes/swivel.stl" />
+				<mesh filename="package://p3dx_description_mod/meshes/swivel.stl" />
 			</geometry>
 			<material name="swivel">
@@ -116,5 +116,5 @@
 			<origin xyz="0 0 0" rpy="0 0 0" />
 			<geometry name="pioneer_geom">
-				<mesh filename="package://p3dx_description/meshes/center_hubcap.stl" />
+				<mesh filename="package://p3dx_description_mod/meshes/center_hubcap.stl" />
 			</geometry>
 			<material name="swivel">
@@ -149,5 +149,5 @@
 			<origin xyz="0 0 0" rpy="0 0 0" />
 			<geometry name="pioneer_geom">
-				<mesh filename="package://p3dx_description/meshes/center_wheel.stl" />
+				<mesh filename="package://p3dx_description_mod/meshes/center_wheel.stl" />
 			</geometry>
 			<material name="WheelBlack">
@@ -179,5 +179,5 @@
 			<origin rpy="0 0 0" xyz="0 0 0" />
 			<geometry name="pioneer_geom">
-				<mesh filename="package://p3dx_description/meshes/front_sonar.stl" />
+				<mesh filename="package://p3dx_description_mod/meshes/front_sonar.stl" />
 			</geometry>
 			<material name="SonarYellow">
@@ -207,5 +207,5 @@
 			<origin xyz="0 0 0" rpy="0 0 0" />
 			<geometry>
-				<mesh filename="package://p3dx_description/meshes/lms100.dae" />
+				<mesh filename="package://p3dx_description_mod/meshes/lms100.dae" />
 			</geometry>
 		</visual>

File: p3dx_description/urdf/pioneer3dx_wheel.xacro (robot description, xacro)
@@ -32,5 +32,5 @@
 				<origin xyz="0 0 0" rpy="0 0 0" />
 				<geometry name="pioneer_geom">
-					<mesh filename="package://p3dx_description/meshes/${suffix}_wheel.stl" />
+					<mesh filename="package://p3dx_description_mod/meshes/${suffix}_wheel.stl" />
 				</geometry>
 				<material name="WheelBlack">
@@ -41,5 +41,5 @@
 				<origin xyz="0 0 0" rpy="${-3.1415927/2} 0 0" />
 				<geometry>
-					<!--<mesh filename="package://p3dx_description/meshes/${suffix}_wheel.stl"/> -->
+					<!--<mesh filename="package://p3dx_description_mod/meshes/${suffix}_wheel.stl"/> -->
 					<cylinder radius="0.09" length="0.01" />
 				</geometry>
@@ -62,5 +62,5 @@
 				<origin xyz="0 0 0" rpy="0 0 0" />
 				<geometry name="pioneer_geom">
-					<mesh filename="package://p3dx_description/meshes/${suffix}_hubcap.stl" />
+					<mesh filename="package://p3dx_description_mod/meshes/${suffix}_hubcap.stl" />
 				</geometry>
 				<material name="HubcapYellow">
@@ -75,5 +75,6 @@
 			</collision>
 		</link>
-		<joint name="base_${suffix}_wheel_joint" type="continuous">
+		<!-- <joint name="base_${suffix}_wheel_joint" type="continuous"> -->
+        <joint name="base_link_${suffix}_wheel_joint" type="continuous">
 			<axis xyz="0 1 0" />
 			<anchor xyz="0 0 0" />
@@ -87,6 +88,10 @@
     <transmission name="${parent}_${suffix}_wheel_trans">
       <type>pr2_mechanism_model/SimpleTransmission</type>
-      <joint name="base_${suffix}_wheel_joint" />
-      <actuator name="base_${suffix}_wheel_motor">
+      <!-- <joint name="base_${suffix}_wheel_joint" /> -->
+      <joint name="base_link_${suffix}_wheel_joint"> <!-- joint now requires hardwareInterface element -->
+        <hardwareInterface>EffortJointInterface</hardwareInterface>
+      </joint>
+      <!-- <actuator name="base_${suffix}_wheel_motor"> -->
+      <actuator name="base_link_${suffix}_wheel_motor">
         <hardwareInterface>EffortJointInterface</hardwareInterface>
         <mechanicalReduction>${reflect * 624/35 * 80/19}</mechanicalReduction>

Commit message: fixed collision

File: p3dx_description/urdf/pioneer3dx.xacro (robot description, xacro)
@@ -101,5 +101,5 @@
 			<origin xyz="0 0 0" rpy="0 0 0" />
 			<geometry>
-				<box size="0 0 0" />
+				<box size="0.001 0.001 0.001" />
 			</geometry>
 		</collision>
@@ -135,5 +135,5 @@
 			<origin xyz="0 0 0" rpy="0 0 0" />
 			<geometry>
-				<box size="0 0 0" />
+				<box size="0.001 0.001 0.001" />
 			</geometry>
 		</collision>
@@ -200,5 +200,5 @@
 			<origin rpy="0 0 0" xyz="0 0 0" />
 			<geometry>
-				<box size="0 0 0" />
+				<box size="0.001 0.001 0.001" />
 			</geometry>
 		</collision>
@@ -225,5 +225,5 @@
 			<origin xyz="0 0 0" rpy="0 0 0" />
 			<geometry>
-				<box size="0.1 0.1 0.1" />
+				<box size="0.001 0.001 0.001" />
 			</geometry>
 		</collision>

File: p3dx_description/urdf/pioneer3dx_wheel.xacro (robot description, xacro)
@@ -74,5 +74,5 @@
 				<origin xyz="0 0 0" rpy="0 0 0" />
 				<geometry>
-					<box size="0 0 0" />
+					<box size="0.001 0.001 0.001" />
 				</geometry>
 			</collision>

Commit message: fixed mod issues

File: p3dx_description/urdf/pioneer3dx.xacro (robot description, xacro)
@@ -24,7 +24,7 @@
 <robot name="pioneer3dx" xmlns:xacro="http://ros.org/wiki/xacro">
   <!-- import all gazebo-customization elements, including gazebo colors -->
-  <xacro:include filename="$(find p3dx_description_mod)/urdf/pioneer3dx.gazebo" />
+  <xacro:include filename="$(find p3dx_description)/urdf/pioneer3dx.gazebo" />
   <!-- import the pioneer 3dx's wheels -->
-  <xacro:include filename="$(find p3dx_description_mod)/urdf/pioneer3dx_wheel.xacro" />
+  <xacro:include filename="$(find p3dx_description)/urdf/pioneer3dx_wheel.xacro" />
   <!-- chassis -->
 	<link name="base_link">
@@ -39,5 +39,5 @@
 			<origin xyz="-0.045 0 0.148" rpy="0 0 0" />
 			<geometry name="pioneer_geom">
-				<mesh filename="package://p3dx_description_mod/meshes/chassis.stl" />
+				<mesh filename="package://p3dx_description/meshes/chassis.stl" />
 			</geometry>
 			<material name="ChassisRed">
@@ -63,5 +63,5 @@
 			<origin xyz="0 0 0" rpy="0 0 0" />
 			<geometry name="top_geom">
-				<mesh filename="package://p3dx_description_mod/meshes/top.stl" />
+				<mesh filename="package://p3dx_description/meshes/top.stl" />
 			</geometry>
 			<material name="TopBlack">
@@ -92,5 +92,5 @@
 			<origin xyz="0 0 0" rpy="0 0 0" />
 			<geometry name="pioneer_geom">
-				<mesh filename="package://p3dx_description_mod/meshes/swivel.stl" />
+				<mesh filename="package://p3dx_description/meshes/swivel.stl" />
 			</geometry>
 			<material name="swivel">
@@ -126,5 +126,5 @@
 			<origin xyz="0 0 0" rpy="0 0 0" />
 			<geometry name="pioneer_geom">
-				<mesh filename="package://p3dx_description_mod/meshes/center_hubcap.stl" />
+				<mesh filename="package://p3dx_description/meshes/center_hubcap.stl" />
 			</geometry>
 			<material name="swivel">
@@ -160,5 +160,5 @@
 			<origin xyz="0 0 0" rpy="0 0 0" />
 			<geometry name="pioneer_geom">
-				<mesh filename="package://p3dx_description_mod/meshes/center_wheel.stl" />
+				<mesh filename="package://p3dx_description/meshes/center_wheel.stl" />
 			</geometry>
 			<material name="WheelBlack">
@@ -191,5 +191,5 @@
 			<origin rpy="0 0 0" xyz="0 0 0" />
 			<geometry name="pioneer_geom">
-				<mesh filename="package://p3dx_description_mod/meshes/front_sonar.stl" />
+				<mesh filename="package://p3dx_description/meshes/front_sonar.stl" />
 			</geometry>
 			<material name="SonarYellow">
@@ -219,5 +219,5 @@
 			<origin xyz="0 0 0" rpy="0 0 0" />
 			<geometry>
-				<mesh filename="package://p3dx_description_mod/meshes/lms100.dae" />
+				<mesh filename="package://p3dx_description/meshes/lms100.dae" />
 			</geometry>
 		</visual>

File: p3dx_description/urdf/pioneer3dx_wheel.xacro (robot description, xacro)
@@ -34,5 +34,5 @@
 				<origin xyz="0 0 0" rpy="0 0 0" />
 				<geometry name="pioneer_geom">
-					<mesh filename="package://p3dx_description_mod/meshes/${suffix}_wheel.stl" />
+					<mesh filename="package://p3dx_description/meshes/${suffix}_wheel.stl" />
 				</geometry>
 				<material name="WheelBlack">
@@ -43,5 +43,5 @@
 				<origin xyz="0 0 0" rpy="${-3.1415927/2} 0 0" />
 				<geometry>
-					<!--<mesh filename="package://p3dx_description_mod/meshes/${suffix}_wheel.stl"/> -->
+					<!--<mesh filename="package://p3dx_description/meshes/${suffix}_wheel.stl"/> -->
 					<cylinder radius="0.09" length="0.01" />
 				</geometry>
@@ -65,5 +65,5 @@
 				<origin xyz="0 0 0" rpy="0 0 0" />
 				<geometry name="pioneer_geom">
-					<mesh filename="package://p3dx_description_mod/meshes/${suffix}_hubcap.stl" />
+					<mesh filename="package://p3dx_description/meshes/${suffix}_hubcap.stl" />
 				</geometry>
 				<material name="HubcapYellow">
